File: bmb/v1.0a/bitmagic-basic.kicad_pcb (KiCad board)
At the start: 4 copper layers, 35 x 16 mm, 37 parts, among them IC1 CY7C68013A-56, J1 Conn, P1 pkl_USB_OTG, U1 3.3V, U2 USBLC6-2, U3 IP425x-4-TTL, U4 IP425x-4-TTL, U5 24LC00, U6 IP425x-4-TTL, X1 24MHz

Commit message: Corrected LED and pullup resistor values in V1.0a.
Parts:
- R1: value 2k7 -> 330E
- R8, R9: value 100k -> 150k
Changed lines of the file:
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@@
       (effects (font (size 0.635 0.635) (thickness 0.1)))
     )
-    (fp_text value 2k7 (at 0 1.55) (layer F.Fab)
+    (fp_text value 330E (at 0 1.55) (layer F.Fab)
       (effects (font (size 0.635 0.635) (thickness 0.1)))
     )
@@
       (effects (font (size 0.635 0.635) (thickness 0.1)))
     )
-    (fp_text value 100k (at 1.8 -0.1 180) (layer F.Fab)
+    (fp_text value 150k (at 1.8 -0.1 180) (layer F.Fab)
       (effects (font (size 0.635 0.635) (thickness 0.1)))
     )
@@
       (effects (font (size 0.635 0.635) (thickness 0.1)))
     )
-    (fp_text value 100k (at 1.5 0 180) (layer F.Fab)
+    (fp_text value 150k (at 1.5 0 180) (layer F.Fab)
       (effects (font (size 0.635 0.635) (thickness 0.1)))
     )
@@
   (via (at 22.5 24.5) (size 0.5) (drill 0.3) (layers F.Cu B.Cu) (net 2))
   (via (at 29.4 31) (size 0.5) (drill 0.3) (layers F.Cu B.Cu) (net 2))
+  (via (at 56.2 32) (size 0.5) (drill 0.3) (layers F.Cu B.Cu) (net 2))
+  (via (at 47.4 28.6) (size 0.5) (drill 0.3) (layers F.Cu B.Cu) (net 2))
   (segment (start 26.175 28.7) (end 27.3 28.7) (width 0.15) (layer F.Cu) (net 3))
   (segment (start 27.7 25.55) (end 27.7 26.025) (width 0.15) (layer F.Cu) (net 3))
@@
   (segment (start 41.95 28.35) (end 41.7 28.6) (width 0.15) (layer F.Cu) (net 18))
   (via (at 41.7 28.6) (size 0.5) (drill 0.3) (layers F.Cu B.Cu) (net 18))
-  (via (at 56.2 32) (size 0.5) (drill 0.3) (layers F.Cu B.Cu) (net 2))
-  (via (at 47.4 28.6) (size 0.5) (drill 0.3) (layers F.Cu B.Cu) (net 2))
   (segment (start 46.375 33.05) (end 47.05 33.05) (width 0.15) (layer F.Cu) (net 19))
   (segment (start 47.81 33.81) (end 49.85 33.81) (width 0.15) (layer F.Cu) (net 19))
